File: aloidia-pcb/epd/epd.kicad_pcb (KiCad board)
At the start: 2 copper layers, 19.6 x 38.6 mm, 20 parts, among them J1 FH12-30S-0.5SH(55), J2 01x08 2.54mm Pin Headers

Commit message: Added pin legends
Other:
- board text added: "3.3V"
- board text added: "BUSY"
- board text added: "CS"
- board text added: "DC"
- board text added: "DIN"
- board text added: "GND"
- board text added: "RST"
- board text added: "SCK"
Changed lines of the file:
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@@
   (gr_line (start 164.7 104.8) (end 165.45 106.075) (layer "Edge.Cuts") (width 0.1))
   (gr_line (start 147.95 105.5) (end 147.95 68.9) (layer "Edge.Cuts") (width 0.1))
+  (gr_text "CS" (at 159.02 71.8 90) (layer "B.SilkS")
+    (effects (font (size 1 1) (thickness 0.15)) (justify left mirror))
+  )
+  (gr_text "GND" (at 148.86 71.8 90) (layer "B.SilkS")
+    (effects (font (size 1 1) (thickness 0.15)) (justify left mirror))
+  )
+  (gr_text "SCK" (at 156.48 71.8 90) (layer "B.SilkS")
+    (effects (font (size 1 1) (thickness 0.15)) (justify left mirror))
+  )
+  (gr_text "3.3V" (at 151.4 71.8 90) (layer "B.SilkS")
+    (effects (font (size 1 1) (thickness 0.15)) (justify left mirror))
+  )
+  (gr_text "DC" (at 161.56 71.8 90) (layer "B.SilkS")
+    (effects (font (size 1 1) (thickness 0.15)) (justify left mirror))
+  )
+  (gr_text "DIN" (at 153.94 71.8 90) (layer "B.SilkS")
+    (effects (font (size 1 1) (thickness 0.15)) (justify left mirror))
+  )
+  (gr_text "BUSY" (at 166.64 71.8 90) (layer "B.SilkS")
+    (effects (font (size 1 1) (thickness 0.15)) (justify left mirror))
+  )
+  (gr_text "RST" (at 164.1 71.8 90) (layer "B.SilkS")
+    (effects (font (size 1 1) (thickness 0.15)) (justify left mirror))
+  )
   (gr_text "19.6" (at 157.65 110.5) (layer "Cmts.User")
     (effects (font (size 1 1) (thickness 0.15)))
