File: aloidia-pcb/solar/solar.kicad_pcb (KiCad board)
At the start: 2 copper layers, 132 x 13.8 mm, 6 parts, among them J1 S2B-PH-SM4-TB(LF)(SN)

Commit message: Added solar breakout module outline dimensions
Other:
- board text added: "13.8"
- board text added: "132"
Changed lines of the file:
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@@
   (gr_line (start 168.25 87.5) (end 169.25 87.5) (layer "B.SilkS") (width 0.1))
   (gr_line (start 168.75 83) (end 168.75 82) (layer "B.SilkS") (width 0.1))
+  (gr_line (start 222.8 91.95) (end 219.85 91.95) (layer "Cmts.User") (width 0.08))
+  (gr_line (start 222.8 78.05) (end 219.8 78.05) (layer "Cmts.User") (width 0.08))
+  (gr_line (start 221.8 91.9) (end 222.6 91.1) (layer "Cmts.User") (width 0.15))
+  (gr_line (start 221.8 78.1) (end 221 78.9) (layer "Cmts.User") (width 0.15))
+  (gr_line (start 87.8 93.9) (end 88.6 93.1) (layer "Cmts.User") (width 0.15))
+  (gr_line (start 221.8 91.9) (end 221 91.1) (layer "Cmts.User") (width 0.15))
+  (gr_line (start 87.8 93.9) (end 88.6 94.7) (layer "Cmts.User") (width 0.15))
+  (gr_line (start 219.85 95) (end 219.85 91.95) (layer "Cmts.User") (width 0.08))
+  (gr_line (start 219.8 93.9) (end 219 94.7) (layer "Cmts.User") (width 0.15))
+  (gr_line (start 87.8 93.9) (end 219.8 93.9) (layer "Cmts.User") (width 0.15))
+  (gr_line (start 221.8 78.1) (end 222.6 78.9) (layer "Cmts.User") (width 0.15))
+  (gr_line (start 221.8 91.9) (end 221.8 78.1) (layer "Cmts.User") (width 0.15))
+  (gr_line (start 219.8 93.9) (end 219 93.1) (layer "Cmts.User") (width 0.15))
+  (gr_line (start 87.75 94.9) (end 87.75 91.9) (layer "Cmts.User") (width 0.08))
   (gr_line (start 170.7 91.9) (end 179.525 91.9) (layer "Edge.Cuts") (width 0.1))
   (gr_line (start 126.9 78.1) (end 136.9 78.1) (layer "Edge.Cuts") (width 0.1))
@@
   (gr_line (start 87.8 78.1) (end 93.1 78.1) (layer "Edge.Cuts") (width 0.1))
   (gr_line (start 93.1 91.9) (end 95.6 89.4) (layer "Edge.Cuts") (width 0.1))
+  (gr_text "13.8" (at 224.1 85) (layer "Cmts.User")
+    (effects (font (size 1 1) (thickness 0.15)))
+  )
+  (gr_text "132" (at 153.9 95.05) (layer "Cmts.User")
+    (effects (font (size 1 1) (thickness 0.15)))
+  )
   (segment (start 215.292893 85) (end 169.157106 85) (width 0.65) (layer "B.Cu") (net 1))
   (segment (start 216.5 85.5) (end 217 86) (width 0.65) (layer "B.Cu") (net 1))
