File: aloidia-pcb/aloidia-right/aloidia-right.kicad_sch (KiCad schematic)
At the start: 225 parts, among them J1 SWD_02x05_1.27mm, J10 Pin headers 2.54mm 01x02, J11 USB4105-GF-A-120, J12 Pin headers 2.54mm 01x08, J2 Pin headers 2.54mm 01x08, J3 SM06B-SRSS-TB, J4 SM03B-SRSS-TB(LF)(SN), J5 S2B-PH-SM4-TB(LF)(SN), J6 Pin headers 2.54mm 01x03, J7 USB4105-GF-A-120, J9 S2B-PH-SM4-TB(LF)(SN), Q1 PJA3404, Q2 DMG9926UDM, Q3 Si2371EDS, Q4 Si2371EDS, Q5 PJA3404, SW1 SSSS213100, SW100 MX_EC11, SW101 SW_Push, SW102 SW_Push, SW103 SW_Push, SW104 SW_Push, SW105 SW_Push, SW106 SW_Push, SW107 SW_Push, SW108 SW_Push, SW110 SW_Push, SW111 SW_Push, SW112 SW_Push, SW113 SW_Push, SW114 SW_Push, SW115 SW_Push, SW116 SW_Push, SW117 SW_Push, SW120 SW_Push, SW121 SW_Push, SW122 SW_Push, SW123 SW_Push, SW124 SW_Push, SW125 SW_Push, SW126 SW_Push, SW127 SW_Push, SW130 SW_Push, SW131 SW_Push, SW132 SW_Push, SW133 SW_Push, SW134 SW_Push, SW135 SW_Push, SW136 SW_Push, SW137 SW_Push, SW140 SW_Push, SW141 SW_Push, SW142 SW_Push, SW143 SW_Push, SW144 SW_Push, SW145 SW_Push, SW146 SW_Push, SW2 MX_EVQWGD001, SW243 SW_Push, SW244 SW_Push, SW246 SW_Push, SW4 EG6201, U1 MAX17048, U2 MDBT50Q-1MV2, U3 MCP1812AT-033/TT, U4 DMN2004DMK-7, U5 BQ24075RGT, U6 AP9101CK6-ANTRG1, U7 STS234050UL30, U8 BQ25504, U9 LTC4359-MS8, Y1 32.768kHz

Commit message: FInished routing right side
Parts:
- removed D108, D116, D126, D136, D140, D146: 1N4148W, Diode_SMD:D_SOD-123, symbol Diode:1N4148W
- removed D11: IN-P32TRRRGB, 0_various:IN-P32TRRRGB, symbol Device:LED_BGRA
- removed H5, H6: 3.2mm_M3, MountingHole:MountingHole_3.2mm_M3_Pad, symbol Mechanical:MountingHole
- removed J9: S2B-PH-SM4-TB(LF)(SN), Connector_JST:JST_PH_S2B-PH-SM4-TB_1x02-1MP_P2.00mm_Horizontal, symbol Connector_Generic:Conn_01x02
- removed S146: MX_stab, marbastlib-mx:STAB_MX_2.25u, symbol marbastlib-mx:MX_stab
- removed S246: MX_stab, marbastlib-mx:STAB_MX_2.75u, symbol marbastlib-mx:MX_stab
- removed SW108, SW116, SW126, SW136, SW140, SW146, SW243, SW246: SW_Push, 0_mx:MX_HS_AS_1u, symbol Switch:SW_Push
- removed SW244: SW_Push, 0_mx:MX_HS_AS_1.25u, symbol Switch:SW_Push
- added D100, D118, D128, D138, D147, D148: 1N4148W, Diode_SMD:D_SOD-123, symbol Diode:1N4148W
- added J9: SM04B-SRSS-TB(LF)(SN), Connector_JST:JST_SH_SM04B-SRSS-TB_1x04-1MP_P1.00mm_Horizontal, symbol Connector_Generic:Conn_01x04
- added S107: MX_stab, marbastlib-mx:STAB_MX_2u, symbol marbastlib-mx:MX_stab
- added S127: MX_stab, marbastlib-mx:STAB_MX_2.25u, symbol marbastlib-mx:MX_stab
- added SW100, SW118, SW128, SW138, SW147, SW148, SW241: SW_Push, 0_mx:MX_HS_AS_1u, symbol Switch:SW_Push
- J12, J2: value Pin headers 2.54mm 01x08 -> SM08B-SRSS-TB(LF)(SN); footprint 0_various:e-Paper Display -> Connector_JST:JST_SH_SM08B-SRSS-TB_1x08-1MP_P1.00mm_Horizontal
- J5: value S2B-PH-SM4-TB(LF)(SN) -> Picoblade 0532614002; footprint Connector_JST:JST_PH_S2B-PH-SM4-TB_1x02-1MP_P2.00mm_Horizontal -> Connector_Molex:Molex_PicoBlade_53261-0271_1x02-1MP_P1.25mm_Horizontal; Digikey ref (none) -> 900-0532614002CT-ND; Manufacturer ref (none) -> 0532614002
- S241: renamed from S132; footprint marbastlib-mx:STAB_MX_2.25u -> marbastlib-mx:STAB_MX_2.75u
- SW112, SW144: footprint 0_mx:MX_HS_AS_1.5u -> 0_mx:MX_HS_AS_1u
- SW117: footprint 0_mx:MX_HS_AS_1u -> 0_mx:MX_HS_AS_1.5u
- SW122: footprint 0_mx:MX_HS_AS_1.75u -> 0_mx:MX_HS_AS_1u
- SW135, SW141: footprint 0_mx:MX_HS_AS_1u -> 0_mx:MX_HS_AS_1.75u
- SW142, SW143: footprint 0_mx:MX_HS_AS_1.25u -> 0_mx:MX_HS_AS_1u
- renumbered D100 to D108, D106 to D116, D147 to D140, SW100 to SW108, SW106 to SW116, SW2 to SW140, SW4 to SW2
Connections:
- net BUSY: now also U2.16 (P0.27); no longer U2.46 (P0.22)
- net CELL+: now also J9.1 (Pin_1), J9.2 (Pin_2)
- net COL0: now also SW140.S1, SW2.3, U2.43 (P0.21), SW100.2; no longer SW108.S2, U2.39 (P0.15)
- net COL1: now also SW141.1, U2.44 (P0.20), SW241.2; no longer SW141.2, U2.38 (P0.16)
- net COL2: now also U2.45 (P0.23); no longer U2.37 (P0.13)
- net COL3: now also SW143.2, U2.42 (P0.19); no longer SW143.1, U2.36 (P0.14)
- net COL4: now also SW144.2, U2.41 (P0.17); no longer SW144.1, U2.13 (P0.28/AIN4)
- net COL6: now also U2.13 (P0.28/AIN4); no longer U2.12 (P0.31/AIN7)
- net COL7: now also U2.12 (P0.31/AIN7), SW147.2; no longer SW140.S2, SW2.3, U2.11 (P0.02/AIN0)
- net COL8: now also SW108.S2, U2.11 (P0.02/AIN0), SW118.2, SW128.2, SW138.2, SW148.2; no longer U2.10 (P0.29/AIN5)
- net COL9: now also U2.46 (P0.22); no longer U2.4 (P1.11)
- net CS: now also U2.21 (P0.05/AIN3); no longer U2.43 (P0.21)
- net D+: now also U7.3 (IO2); no longer U7.1 (IO1)
- net D-: now also U7.4 (IO3); no longer U7.6 (IO4)
- net DC: now also U2.20 (P0.04/AIN2); no longer U2.44 (P0.20)
- net DIN: now also U2.23 (TRACECLK/P0.07); no longer U2.41 (P0.17)
- net EC_ENCA: now also U2.5 (P1.12); no longer U2.48 (P0.24)
- net EC_ENCB: now also U2.4 (P1.11); no longer U2.49 (P0.25)
- net EVQ_ENCA: now also SW2.9, U2.38 (P0.16); no longer SW2.12, U2.24 (P0.08)
- net EVQ_ENCB: now also SW2.12, U2.37 (P0.13); no longer SW2.9, U2.22 (P0.06)
- net GND: now also J9.3 (Pin_3), J9.4 (Pin_4)
- net ROW0: now also U2.10 (P0.29/AIN5), D100.2 (A); no longer D116.2 (A), U2.9 (P0.03/AIN1)
- net ROW1: now also D116.2 (A), U2.9 (P0.03/AIN1), D118.2 (A); no longer U2.8 (P1.15)
- net ROW2: now also U2.8 (P1.15), D128.2 (A); no longer U2.7 (P1.14)
- net ROW3: now also U2.7 (P1.14), D138.2 (A); no longer U2.6 (P1.13)
- net ROW4: now also U2.6 (P1.13), D147.2 (A), D148.2 (A); no longer U2.5 (P1.12)
- net ROW4_SW: now also SW140.S2; no longer SW140.S1
- net RST: now also U2.19 (P0.26); no longer U2.45 (P0.23)
- net SCK: now also U2.22 (P0.06); no longer U2.42 (P0.19)
- net at D144.1 (K): now also SW144.1; no longer SW144.2
- net at D141.1 (K): now also SW141.2, SW241.1; no longer SW141.1
- net at D143.1 (K): now also SW143.1; no longer SW143.2
- new net: D128.1 (K), SW128.1
- new net: D147.1 (K), SW147.1
- new net: D118.1 (K), SW118.1
- new net: D138.1 (K), SW138.1
- new net: D100.1 (K), SW100.1
- new net: D148.1 (K), SW148.1
- no-connect marks 34 -> 28
Other:
- note removed: "20431"
- note removed: "Do not populate 5.1k resistors if using daugtherboard"
- title: ALOIDIA Keyboard Left Side -> ALOIDIA Keyboard Right Side
- moved on the sheet: D116, D140, D8, S241, SW116
